File: cesar-3.kicad_pcb (KiCad board)
At the start: 2 copper layers, 85 parts, among them U1 Nice_Nano_V2

Commit message: after rotarion
Parts:
- moved D36 46.6 mm to (363.2, 91.5), turned to 111 degrees
- moved D24 43.9 mm to (356.9, 75.1), turned to 111 degrees
- moved S25 43.3 mm to (73.9, 92.8), turned to -14 degrees
- moved S36 43.2 mm to (354.0, 89.3), turned to 21 degrees
- moved D12 41.8 mm to (350.2, 57.6), turned to 111 degrees
- moved S13 41.2 mm to (78.4, 74.4), turned to -14 degrees
- moved D25 41.2 mm to (80.8, 99.1), turned to 76 degrees
- moved D35 41.1 mm to (346.2, 99.0), turned to 111 degrees
- moved S24 40.4 mm to (347.2, 71.6), turned to 21 degrees
- moved S1 40.2 mm to (83.0, 55.9), turned to -14 degrees
- moved D13 38.8 mm to (85.1, 81.8), turned to 76 degrees
- moved S12 38.5 mm to (340.4, 53.9), turned to 21 degrees
- moved D23 37.7 mm to (339.6, 81.8), turned to 111 degrees
- moved D1 37.5 mm to (89.1, 65.9), turned to 76 degrees
- moved S35 37.3 mm to (336.3, 96.1), turned to 21 degrees
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
Commit message: before rotation
Parts:
- moved D36 50.8 mm to (348.2, 140.0), turned to 83 degrees
- moved D24 48.0 mm to (350.4, 122.7), turned to 83 degrees
- moved D12 46.5 mm to (352.7, 104.1), turned to 83 degrees
- moved S36 46.4 mm to (341.2, 133.9), turned to -7 degrees
- moved S24 43.6 mm to (343.5, 115.0), turned to -7 degrees
- moved S25 43.4 mm to (87.7, 133.9), turned to 7 degrees
- moved D35 43.0 mm to (329.8, 138.8), turned to 83 degrees
- moved S12 42.6 mm to (345.8, 96.2), turned to -7 degrees
- moved D25 41.3 mm to (96.5, 137.3), turned to 97 degrees
- moved S13 41.3 mm to (85.4, 115.0), turned to 7 degrees
- moved S1 40.2 mm to (83.1, 96.2), turned to 7 degrees
- moved D23 39.4 mm to (332.0, 120.4), turned to 83 degrees
- moved D13 38.9 mm to (94.3, 119.6), turned to 97 degrees
- moved S35 38.1 mm to (322.3, 131.6), turned to -7 degrees
- moved D11 37.6 mm to (334.1, 103.0), turned to 83 degrees
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Routing:
- net row0: track 245.8 -> 255.2 mm
- net row1: track 249.2 -> 258.1 mm
- net row2: track 284.1 -> 291.5 mm
- net col11: track 157.1 -> 161.7 mm
- net col10: track 140.8 -> 145.2 mm

Commit message: after rotation
Routing:
- net row1: track 258.1 -> 270.4 mm
- net row2: track 291.5 -> 302.7 mm
- net row3: track 190.3 -> 199.4 mm

Commit message: valid after rotation
Parts:
- moved D36 46.8 mm to (363.8, 95.9), turned to 104 degrees
- moved D24 44.7 mm to (359.6, 78.9), turned to 104 degrees
- moved S25 43.5 mm to (73.9, 92.7), turned to -14 degrees
- moved S36 43.5 mm to (355.0, 92.7), turned to 14 degrees
- moved D12 43.4 mm to (355.1, 60.7), turned to 104 degrees
- moved D25 41.4 mm to (80.8, 99.0), turned to 76 degrees
- moved S13 41.4 mm to (78.5, 74.2), turned to -14 degrees
- moved S24 41.4 mm to (350.4, 74.2), turned to 14 degrees
- moved D35 40.9 mm to (346.1, 101.3), turned to 104 degrees
- moved S1 40.4 mm to (83.1, 55.8), turned to -14 degrees
- moved S12 40.4 mm to (345.8, 55.8), turned to 14 degrees
- moved D13 39.0 mm to (85.1, 81.7), turned to 76 degrees
- moved D23 38.3 mm to (341.6, 83.4), turned to 104 degrees
- moved D1 37.7 mm to (89.1, 65.8), turned to 76 degrees
- moved S26 37.1 mm to (92.3, 97.3), turned to -14 degrees
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
Commit message: routing complete
Parts:
- moved U1 92.3 mm to (214.4, 94.0)
Routing:
- net row3: track 199.4 -> 272.0 mm
- net row2: track 302.7 -> 374.7 mm
- net row1: track 270.4 -> 339.1 mm
- net row0: track 255.1 -> 323.6 mm
- net col5: track 98.1 -> 123.8 mm
- net col6: track 85.7 -> 110.1 mm
- net col4: track 116.3 -> 140.3 mm
- net col7: track 106.4 -> 129.7 mm
- net col3: track 135.9 -> 158.9 mm
- net col0: track 178.1 -> 200.6 mm
- net col2: track 129.7 -> 151.8 mm
- net col1: track 159.2 -> 180.8 mm
- net col11: track 161.7 -> 183.1 mm
- net col8: track 129.7 -> 151.0 mm
- net col10: track 145.2 -> 166.1 mm
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Other:
- board outline added: 304.2 x 117.9 mm

Commit message: Production v0.1 PCB and plate dxf files
The v0.1 prototype and the dxf files corresponding to the bottom and top
plates.
Parts:
- added ?: , , F.Cu at (73.0, 102.1)
- added ?: , , F.Cu at (297.6, 133.1)
- added ?: , , F.Cu at (107.0, 133.6)
- added ?: , , F.Cu at (156.9, 98.1)
- added ?: , , F.Cu at (246.9, 97.3)
- added ?: , , F.Cu at (156.0, 149.9)
- added ?: , , F.Cu at (331.1, 102.1)
- added ?: , , F.Cu at (77.6, 83.6)
- added ?: , , F.Cu at (248.2, 150.0)
- added ?: , , F.Cu at (326.5, 83.6)
- added D0: IR26-21C_L110_TR8, LED_SMD:LED_1206_3216Metric, F.Cu at (195.6, 109.2)
- added D43: IR26-21C_L110_TR8, LED_SMD:LED_1206_3216Metric, F.Cu at (203.2, 109.2)
- added R0: 4k7, Resistor_SMD:R_0805_2012Metric, F.Cu at (199.4, 111.8)
- added R1: 4k7, Resistor_SMD:R_0805_2012Metric, F.Cu at (207.0, 111.8)
- added SW0: SW_Push, Button_Switch_SMD:SW_Tactile_SPST_NO_Straight_CK_PTS636Sx25SMTRLFS, F.Cu at (180.9, 97.5)
- moved S24 20.5 mm to (338.0, 90.5)
- moved S18 20.5 mm to (160.5, 115.4)
- moved S28 20.5 mm to (121.8, 110.2)
- moved D27 20.5 mm to (108.0, 116.1)
- moved S40 20.5 mm to (244.2, 162.1)
- moved D22 20.5 mm to (305.9, 95.5)
- moved D24 20.5 mm to (347.2, 95.2)
- moved S19 20.5 mm to (243.6, 115.4)
- moved S5 20.5 mm to (150.6, 88.1)
- moved S17 20.5 mm to (143.8, 105.8)
- moved S12 20.5 mm to (333.4, 72.1)
- moved D31 20.5 mm to (260.3, 135.8)
- moved S22 20.5 mm to (295.8, 92.2)
- moved D29 20.5 mm to (141.8, 134.0)
- moved D42 20.5 mm to (291.3, 141.1)
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Connections:
- U1 pad 1: unconnected-(U1-D1-Pad1) -> Net-(D43-A)
- U1 pad 2: unconnected-(U1-D0-Pad2) -> Net-(D0-A)
- U1 pad 22: unconnected-(U1-RST-Pad22) -> Net-(U1-RST)
- U1 pad 23: unconnected-(U1-GND-Pad23) -> Net-(SW0-Pad1)
- U1 pad 4: unconnected-(U1-GND-Pad4) -> Net-(R0-Pad1)
Routing:
- net Net-(R0-Pad1): track 0.00 -> 36.6 mm
- net Net-(U1-RST): track 0.00 -> 31.3 mm
- net Net-(D43-A): track 0.00 -> 26.2 mm, vias 0 -> 1
- net Net-(SW0-Pad1): track 0.00 -> 23.6 mm
- net col5: track 123.8 -> 146.4 mm
- net col11: track 183.1 -> 204.4 mm, vias 3 -> 4
- net Net-(D0-A): track 0.00 -> 17.7 mm, vias 0 -> 1
- net col10: track 166.1 -> 182.7 mm, vias 3 -> 4
- net col4: track 140.3 -> 156.7 mm
- net col9: track 136.0 -> 152.2 mm, vias 3 -> 4
- net col3: track 158.9 -> 173.6 mm
- net col8: track 151.0 -> 165.4 mm, vias 4 -> 5
- net row0: track 323.6 -> 336.9 mm
- net col2: track 151.8 -> 164.7 mm
- net col1: track 180.8 -> 192.1 mm
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Other:
- outline, holes or cut-outs redrawn
