File: cesar-3.kicad_sch (KiCad schematic)
At the start: 85 parts, among them U1 Nice_Nano_V2

Commit message: Production v0.1 PCB and plate dxf files
The v0.1 prototype and the dxf files corresponding to the bottom and top
plates.
Parts:
- added D0, D43: IR26-21C_L110_TR8, LED_SMD:LED_1206_3216Metric, symbol LED:IR26-21C_L110_TR8
- added R0, R1: 4k7, Resistor_SMD:R_0805_2012Metric, symbol Device:R
- added SW0: SW_Push, Button_Switch_SMD:SW_Tactile_SPST_NO_Straight_CK_PTS636Sx25SMTRLFS, symbol Switch:SW_Push
Connections:
- net at U1.1 (D1): now also D43.2 (A)
- net at U1.2 (D0): now also D0.2 (A)
- net at U1.22 (RST): now also SW0.2
- net at U1.23 (GND): now also SW0.1
- net at U1.4 (GND): now also R0.1, R1.1
- new net: D0.1 (K), R0.2
- new net: D43.1 (K), R1.2
